Commit message: version 1

File: src/husky/husky_description/urdf/accessories/zed2.urdf.xacro (robot description, xacro)
@@ -21,4 +21,9 @@
           <mesh filename="package://husky_description/meshes/accessories/ZED2i.stl" scale="0.001 0.001 0.001"/>
         </geometry>
+        <material
+        name="">
+        <color
+          rgba="0.15 0.15 0.15 1" />
+      </material>
       </visual>
     </link>

File: src/husky/husky_description/urdf/decorations.urdf.xacro (robot description, xacro)
@@ -84,4 +84,9 @@
           <mesh filename="package://husky_description/meshes/reachrs2.stl" scale="0.03 0.03 0.03" />
         </geometry>
+        <material
+        name="">
+        <color
+          rgba="0.3 0.3 0.3 1" />
+      </material>
       </visual>
     </link>

File: src/husky/husky_description/urdf/husky_macro.urdf.xacro (robot description, xacro)
@@ -62,5 +62,5 @@
       <parent link="${prefix}top_structure"/>
       <child link="${prefix}zed2_camera_center"/>
-      <origin xyz="-0.35 -0.2 0.309" rpy="0 0 0"/>
+      <origin xyz="-0.839 0.2 0.293" rpy="0 0 ${M_PI}"/>
     </joint>
     <xacro:zed2 link_prefix="${prefix}"
@@ -103,4 +103,5 @@
       <child link="${prefix}gps_link" />
     </joint>
+    <!-- Top Structure-->
     <link name="top_structure">
     <inertial>

File: src/livox_laser_simulation_ros2/urdf/HAP.xacro (robot description, xacro)
@@ -28,4 +28,9 @@
             <mesh filename="package://husky_description/meshes/accessories/HAP.stl" scale="0.001 0.001 0.001"/>
         </geometry>
+        <material
+        name="">
+        <color
+          rgba="0.05 0.05 0.05 1" />
+      </material>
   </visual>
 </link>
